File: hardware/kicad/reflow.kicad_sch (KiCad schematic)
At the start: 35 parts, among them J1 24V_IN, J2 HEATER, J3 MAX31855, J4 OLED, Q1 IRFS4710, Q2 BS170, Q3 BS170, SW1 ENC, SW2 START, U2 LM2575-ADJ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

Commit message: hardware: BOM generated and cross-checked against DTU component shop
Add check_bom_against_shop.py: reads board-soldered parts from the netlist
(excludes A1/J3/J4 modules + F1 fuse holder), normalises each value (µ/u, Ω/R,
k/K, E96 codes, cap/diode formats) and asserts a Part_Number/Value match in
dtu_component_shop(1).csv. Exit 0 = all resolve.

Snap the parts that only differed by value-string formatting to shop stock:
D3 24V-rail TVS -> P6KE24P (24V standoff, ~33V clamp < 35V caps), D4 drain TVS
-> 1.5KE36A (36V standoff > 24V rail, ~52V clamp << Q1 100V Vds), J1/J2 ->
2 pol skrueterminal, SW1 -> Rotary 1x12 EYE, SW2 -> Pushbutton, D1 -> LED 5MM
GRØN. All 31 board parts now resolve.

Add docs/BOM.md: board-parts table (every line maps to a shop Part_Number) +
consolidated purchase list + External/bring-your-own section (ESP32 DevKit,
MAX31855+thermocouple, SSD1306 OLED, 24V PSU, PTC plate, thermal fuse, 24V
fuse holder). ERC=0, pad-nets/boot-safety/net-contract still pass.
Parts:
- D1: value STATUS -> LED 5MM GRØN
- D3: value SMBJ26A -> P6KE24P
- D4: value SMBJ33A -> 1.5KE36A
- F1: value 15A -> 15A (holder, BYO)
- J1: value 24V_IN -> 2 pol skrueterminal
- J2: value HEATER -> 2 pol skrueterminal
- SW1: value ENC -> Rotary 1x12 EYE
- SW2: value START -> Pushbutton
Changed lines of the file:
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@@
 			)
 		)
-		(property "Value" "24V_IN"
+		(property "Value" "2 pol skrueterminal"
 			(at 35.08 42.54 0)
 			(effects
@@
 			)
 		)
-		(property "Value" "15A"
+		(property "Value" "15A (holder, BYO)"
 			(at 60.08 42.54 0)
 			(effects
@@
 			)
 		)
-		(property "Value" "SMBJ26A"
+		(property "Value" "P6KE24P"
 			(at 80.08 52.54 0)
 			(effects
@@
 			)
 		)
-		(property "Value" "HEATER"
+		(property "Value" "2 pol skrueterminal"
 			(at 385.08 202.54 0)
 			(effects
@@
 			)
 		)
-		(property "Value" "SMBJ33A"
+		(property "Value" "1.5KE36A"
 			(at 360.08 197.54 0)
 			(effects
@@
 			)
 		)
-		(property "Value" "ENC"
+		(property "Value" "Rotary 1x12 EYE"
 			(at 335.08 92.54 0)
 			(effects
@@
 			)
 		)
-		(property "Value" "START"
+		(property "Value" "Pushbutton"
 			(at 335.08 132.54 0)
 			(effects
@@
 			)
 		)
-		(property "Value" "STATUS"
+		(property "Value" "LED 5MM GRØN"
 			(at 385.08 132.54 0)
 			(effects
